File: TRS NANO.sch (EAGLE design)
At the start: 29 parts, among them M1 ARDUINO-NANO-3.0, Q5 BC548, Q6 BC548, Q7 BC548, Q8 BC548, T1 351, T2 LM35, T3 351, T41 351, T42 351

Commit message: PDFs
Parts:
- renumbered S1 to MIN, S2 to MAX
Changed lines of the file:
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@@
 <part name="D7" library="diode" deviceset="DIODE-" device="D-7.5" value="4007"/>
 <part name="D8" library="diode" deviceset="DIODE-" device="D-7.5" value="4007"/>
-<part name="S1" library="switch-omron" deviceset="10-XX" device=""/>
-<part name="S2" library="switch-omron" deviceset="10-XX" device=""/>
+<part name="MIN" library="switch-omron" deviceset="10-XX" device=""/>
+<part name="MAX" library="switch-omron" deviceset="10-XX" device=""/>
 <part name="SUPPLY2" library="supply2" deviceset="GND" device=""/>
 <part name="SUPPLY4" library="supply2" deviceset="GND" device=""/>
@@
 <instance part="D7" gate="G$1" x="-16.51" y="107.95"/>
 <instance part="D8" gate="G$1" x="-26.67" y="107.95"/>
-<instance part="S1" gate="1" x="5.08" y="46.99" rot="R270"/>
-<instance part="S2" gate="1" x="30.48" y="46.99" rot="R270"/>
+<instance part="MIN" gate="1" x="5.08" y="46.99" rot="R270"/>
+<instance part="MAX" gate="1" x="30.48" y="46.99" rot="R270"/>
 <instance part="SUPPLY2" gate="GND" x="-19.05" y="73.66"/>
 <instance part="SUPPLY4" gate="GND" x="10.16" y="29.21" rot="MR0"/>
@@
 </segment>
 <segment>
-<pinref part="S1" gate="1" pin="P1"/>
-<pinref part="S1" gate="1" pin="P"/>
+<pinref part="MIN" gate="1" pin="P1"/>
+<pinref part="MIN" gate="1" pin="P"/>
 <wire x1="0" y1="46.99" x2="0" y2="44.45" width="0.1524" layer="91"/>
 <pinref part="SUPPLY11" gate="+5V" pin="+5V"/>
@@
 </segment>
 <segment>
-<pinref part="S2" gate="1" pin="P1"/>
-<pinref part="S2" gate="1" pin="P"/>
+<pinref part="MAX" gate="1" pin="P1"/>
+<pinref part="MAX" gate="1" pin="P"/>
 <wire x1="25.4" y1="46.99" x2="25.4" y2="44.45" width="0.1524" layer="91"/>
 <pinref part="SUPPLY3" gate="+5V" pin="+5V"/>
@@
 </segment>
 <segment>
-<pinref part="S1" gate="1" pin="S"/>
+<pinref part="MIN" gate="1" pin="S"/>
 <wire x1="11.43" y1="46.99" x2="10.16" y2="46.99" width="0.1524" layer="91"/>
-<pinref part="S1" gate="1" pin="S1"/>
+<pinref part="MIN" gate="1" pin="S1"/>
 <wire x1="10.16" y1="44.45" x2="10.16" y2="46.99" width="0.1524" layer="91"/>
 <junction x="10.16" y="46.99"/>
@@
 </segment>
 <segment>
-<pinref part="S2" gate="1" pin="S1"/>
-<pinref part="S2" gate="1" pin="S"/>
+<pinref part="MAX" gate="1" pin="S1"/>
+<pinref part="MAX" gate="1" pin="S"/>
 <wire x1="35.56" y1="44.45" x2="35.56" y2="46.99" width="0.1524" layer="91"/>
 <wire x1="36.83" y1="46.99" x2="35.56" y2="46.99" width="0.1524" layer="91"/>

Commit message: elimina LM35
Parts:
- removed MAX, MIN: (no value), switch-omron:10-XX
- removed T2: LM35, transistor-neu-to92:-NPN-TO92-CBE
- added J1: (no value), jumper:JP2W
Connections:
- net +5V: now also J1.2, X3-3.KL; no longer MAX.P, MAX.P1, MIN.P, MIN.P1, T2.C, X3-2.KL
- net A0: now also J1.3; no longer MIN.S, MIN.S1
- net A1: now also J1.1, R1.2; no longer MAX.S, MAX.S1, R1.1
- net A4: now also X3-1.KL; no longer T2.B
- net A7: now also X3-2.KL; no longer X3-1.KL
- net GND: now also R1.1, T413.O; no longer R1.2, T2.E, T412.O, X3-3.KL
- net T41: now also T412.O; no longer T413.O
Other:
- moved on the sheet: R1

Commit message: update
Parts:
- removed X3: (no value), con-ptr500:AK500/4
- added IC: LM35, transistor-npn:BC548
- added R3: 500K, rcl:R-EU_0207/7
- added R4: 1M, rcl:R-EU_0207/15
- added SL2: (no value), con-amp-quick:M03
- added X1, X2: (no value), con-ptr500:AK500/2
Connections:
- removed net A4: M1.A4, X3-1.KL
- removed net A7: M1.A7, X3-2.KL
- new net LM35_S: IC.B, M1.A6
- new net RX: M1.D0/TXD, SL2.1
- new net TEMP_S: M1.A7, R3.2, R4.1
- new net TRIM_A: M1.A4, X1-1.KL
- new net TRIM_B: M1.A3, X1-2.KL
- new net TX: M1.D1/RXD, SL2.2
- net +5V: now also IC.C, X2-2.KL; no longer X3-3.KL
- net GND: now also IC.E, R3.1, SL2.3, X2-1.KL; no longer M1.A3, M1.A6, X3-4.KL
- net TEMP: now also R4.2
Other:
- moved on the sheet: D5, D6, D7, D8, T1, T3, T41, T42

Commit message: Add
Parts:
- removed SL2: (no value), con-amp-quick:M03
- added SV1: (no value), con-lstb:MA04-1
- R1: device rcl:R-EU_0207/7 -> rcl:R-EU_0207/10
- R10, R11, R8, R9: device rcl:R-EU_0207/7 -> rcl:R-EU_0207/5V
Connections:
- net +5V: now also SV1.4
- net A: now also R8.1; no longer R8.2
- net B: now also R9.1; no longer R9.2
- net C: now also R10.1; no longer R10.2
- net D: now also R11.1; no longer R11.2
- net GND: now also SV1.3; no longer SL2.3
- net N$4: now also R9.2; no longer R9.1
- net N$5: now also R10.2; no longer R10.1
- net N$6: now also R11.2; no longer R11.1
- net N$8: now also R8.2; no longer R8.1
- net RX: now also SV1.1; no longer SL2.1
- net TX: now also SV1.2; no longer SL2.2
Other:
- moved on the sheet: R10, R11, R8, R9
Changed lines of the file:
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@@
 <part name="SUPPLY18" library="supply2" deviceset="GND" device=""/>
 <part name="T1" library="relay" deviceset="351" device=""/>
-<part name="R8" library="rcl" deviceset="R-EU_" device="0207/7" value="1k"/>
+<part name="R8" library="rcl" deviceset="R-EU_" device="0207/5V" value="1k"/>
 <part name="SUPPLY19" library="supply2" deviceset="+12V" device=""/>
 <part name="D1" library="diode" deviceset="DIODE-" device="D-7.5" value="4007"/>
 <part name="SUPPLY20" library="supply2" deviceset="GND" device=""/>
 <part name="T3" library="relay" deviceset="351" device=""/>
-<part name="R9" library="rcl" deviceset="R-EU_" device="0207/7" value="1k"/>
+<part name="R9" library="rcl" deviceset="R-EU_" device="0207/5V" value="1k"/>
 <part name="SUPPLY21" library="supply2" deviceset="+12V" device=""/>
 <part name="D2" library="diode" deviceset="DIODE-" device="D-7.5" value="4007"/>
 <part name="SUPPLY22" library="supply2" deviceset="GND" device=""/>
 <part name="T42" library="relay" deviceset="351" device=""/>
-<part name="R10" library="rcl" deviceset="R-EU_" device="0207/7" value="1k"/>
+<part name="R10" library="rcl" deviceset="R-EU_" device="0207/5V" value="1k"/>
 <part name="SUPPLY23" library="supply2" deviceset="+12V" device=""/>
 <part name="D3" library="diode" deviceset="DIODE-" device="D-7.5" value="4007"/>
 <part name="SUPPLY24" library="supply2" deviceset="GND" device=""/>
 <part name="T41" library="relay" deviceset="351" device=""/>
-<part name="R11" library="rcl" deviceset="R-EU_" device="0207/7" value="1k"/>
+<part name="R11" library="rcl" deviceset="R-EU_" device="0207/5V" value="1k"/>
 <part name="SUPPLY25" library="supply2" deviceset="+12V" device=""/>
 <part name="D4" library="diode" deviceset="DIODE-" device="D-7.5" value="4007"/>
@@
 <part name="SUPPLY4" library="supply2" deviceset="GND" device=""/>
 <part name="SUPPLY16" library="supply2" deviceset="GND" device=""/>
-<part name="R1" library="rcl" deviceset="R-EU_" device="0207/7" value="1k"/>
+<part name="R1" library="rcl" deviceset="R-EU_" device="0207/10" value="1k"/>
 <part name="R2" library="rcl" deviceset="R-EU_" device="0207/7" value="1k"/>
 <part name="SUPPLY11" library="supply2" deviceset="+5V" device=""/>
@@
 <part name="SUPPLY15" library="supply2" deviceset="GND" device=""/>
 <part name="SUPPLY27" library="supply2" deviceset="+5V" device=""/>
-<part name="SL2" library="con-amp-quick" deviceset="M03" device=""/>
 <part name="X1" library="con-ptr500" deviceset="AK500/2" device=""/>
 <part name="X2" library="con-ptr500" deviceset="AK500/2" device=""/>
+<part name="SV1" library="con-lstb" deviceset="MA04-1" device=""/>
+<part name="SUPPLY6" library="supply2" deviceset="+5V" device=""/>
 </parts>
 <sheets>
@@
 <instance part="T1" gate="2" x="58.42" y="43.18"/>
 <instance part="T1" gate="3" x="58.42" y="27.94"/>
-<instance part="R8" gate="G$1" x="-62.23" y="-21.59" rot="R270"/>
+<instance part="R8" gate="G$1" x="-59.69" y="-21.59" rot="R90"/>
 <instance part="SUPPLY19" gate="+12V" x="-52.07" y="6.35"/>
 <instance part="D1" gate="G$1" x="-59.69" y="-3.81" rot="R90"/>
@@
 <instance part="T3" gate="2" x="73.66" y="43.18"/>
 <instance part="T3" gate="3" x="73.66" y="27.94"/>
-<instance part="R9" gate="G$1" x="-36.83" y="-21.59" rot="R270"/>
+<instance part="R9" gate="G$1" x="-36.83" y="-21.59" rot="R90"/>
 <instance part="SUPPLY21" gate="+12V" x="-29.21" y="6.35"/>
 <instance part="D2" gate="G$1" x="-36.83" y="-3.81" rot="R90"/>
@@
 <instance part="T42" gate="2" x="88.9" y="43.18"/>
 <instance part="T42" gate="3" x="88.9" y="27.94"/>
-<instance part="R10" gate="G$1" x="-13.97" y="-21.59" rot="R270"/>
+<instance part="R10" gate="G$1" x="-13.97" y="-21.59" rot="R90"/>
 <instance part="SUPPLY23" gate="+12V" x="-6.35" y="6.35"/>
 <instance part="D3" gate="G$1" x="-13.97" y="-3.81" rot="R90"/>
@@
 <instance part="T41" gate="2" x="104.14" y="43.18"/>
 <instance part="T41" gate="3" x="104.14" y="27.94"/>
-<instance part="R11" gate="G$1" x="8.89" y="-21.59" rot="R270"/>
+<instance part="R11" gate="G$1" x="8.89" y="-21.59" rot="R90"/>
 <instance part="SUPPLY25" gate="+12V" x="16.51" y="6.35"/>
 <instance part="D4" gate="G$1" x="8.89" y="-3.81" rot="R90"/>
@@
 <instance part="SUPPLY15" gate="GND" x="48.26" y="-7.62" rot="MR0"/>
 <instance part="SUPPLY27" gate="+5V" x="48.26" y="10.16" rot="MR0"/>
-<instance part="SL2" gate="G$1" x="-57.15" y="40.64" rot="R180"/>
 <instance part="X1" gate="-1" x="-27.94" y="43.18"/>
 <instance part="X1" gate="-2" x="-27.94" y="38.1"/>
 <instance part="X2" gate="-1" x="-27.94" y="33.02"/>
 <instance part="X2" gate="-2" x="-27.94" y="27.94"/>
+<instance part="SV1" gate="1" x="-53.34" y="38.1" rot="R180"/>
+<instance part="SUPPLY6" gate="+5V" x="-63.5" y="46.99"/>
 </instances>
 <busses>
@@
 <segment>
 <pinref part="SUPPLY3" gate="GND" pin="GND"/>
-<pinref part="SL2" gate="G$1" pin="3"/>
-<wire x1="-64.77" y1="38.1" x2="-66.04" y2="38.1" width="0.1524" layer="91"/>
+<pinref part="SV1" gate="1" pin="3"/>
+<wire x1="-60.96" y1="38.1" x2="-66.04" y2="38.1" width="0.1524" layer="91"/>
 </segment>
 <segment>
@@
 <net name="A" class="0">
 <segment>
-<pinref part="R8" gate="G$1" pin="2"/>
-<wire x1="-64.77" y1="-26.67" x2="-62.23" y2="-26.67" width="0.1524" layer="91"/>
-<label x="-64.77" y="-26.67" size="1.778" layer="95" rot="R180" xref="yes"/>
+<label x="-62.23" y="-26.67" size="1.778" layer="95" rot="R180" xref="yes"/>
+<pinref part="R8" gate="G$1" pin="1"/>
+<wire x1="-59.69" y1="-26.67" x2="-62.23" y2="-26.67" width="0.1524" layer="91"/>
 </segment>
 <segment>
@@
 <net name="B" class="0">
 <segment>
-<pinref part="R9" gate="G$1" pin="2"/>
-<wire x1="-39.37" y1="-26.67" x2="-36.83" y2="-26.67" width="0.1524" layer="91"/>
 <label x="-39.37" y="-26.67" size="1.778" layer="95" rot="R180" xref="yes"/>
+<pinref part="R9" gate="G$1" pin="1"/>
+<wire x1="-36.83" y1="-26.67" x2="-39.37" y2="-26.67" width="0.1524" layer="91"/>
 </segment>
 <segment>
@@
 <net name="C" class="0">
 <segment>
-<pinref part="R10" gate="G$1" pin="2"/>
-<wire x1="-16.51" y1="-26.67" x2="-13.97" y2="-26.67" width="0.1524" layer="91"/>
 <label x="-16.51" y="-26.67" size="1.778" layer="95" rot="R180" xref="yes"/>
+<pinref part="R10" gate="G$1" pin="1"/>
+<wire x1="-13.97" y1="-26.67" x2="-16.51" y2="-26.67" width="0.1524" layer="91"/>
 </segment>
 <segment>
@@
 <net name="D" class="0">
 <segment>
-<pinref part="R11" gate="G$1" pin="2"/>
-<wire x1="6.35" y1="-26.67" x2="8.89" y2="-26.67" width="0.1524" layer="91"/>
 <label x="6.35" y="-26.67" size="1.778" layer="95" rot="R180" xref="yes"/>
+<pinref part="R11" gate="G$1" pin="1"/>
+<wire x1="8.89" y1="-26.67" x2="6.35" y2="-26.67" width="0.1524" layer="91"/>
 </segment>
 <segment>
@@
 <wire x1="16.51" y1="-11.43" x2="16.51" y2="-8.89" width="0.1524" layer="91"/>
 <junction x="16.51" y="-8.89"/>
-</segment>
-</net>
-<net name="N$4" class="0">
-<segment>
-<pinref part="R9" gate="G$1" pin="1"/>
-<pinref part="Q6" gate="G$1" pin="B"/>
-<wire x1="-36.83" y1="-16.51" x2="-34.29" y2="-16.51" width="0.1524" layer="91"/>
-</segment>
-</net>
-<net name="N$5" class="0">
-<segment>
-<pinref part="Q7" gate="G$1" pin="B"/>
-<pinref part="R10" gate="G$1" pin="1"/>
-<wire x1="-11.43" y1="-16.51" x2="-13.97" y2="-16.51" width="0.1524" layer="91"/>
-</segment>
-</net>
-<net name="N$6" class="0">
-<segment>
-<pinref part="R11" gate="G$1" pin="1"/>
-<pinref part="Q8" gate="G$1" pin="B"/>
-<wire x1="8.89" y1="-16.51" x2="11.43" y2="-16.51" width="0.1524" layer="91"/>
-</segment>
-</net>
-<net name="N$8" class="0">
-<segment>
-<pinref part="Q5" gate="G$1" pin="B"/>
-<pinref part="R8" gate="G$1" pin="1"/>
-<wire x1="-57.15" y1="-16.51" x2="-62.23" y2="-16.51" width="0.1524" layer="91"/>
 </segment>
 </net>
@@
 <wire x1="-22.86" y1="27.94" x2="-10.16" y2="27.94" width="0.1524" layer="91"/>
 </segment>
+<segment>
+<pinref part="SV1" gate="1" pin="4"/>
+<pinref part="SUPPLY6" gate="+5V" pin="+5V"/>
+<wire x1="-60.96" y1="35.56" x2="-63.5" y2="35.56" width="0.1524" layer="91"/>
+<wire x1="-63.5" y1="35.56" x2="-63.5" y2="44.45" width="0.1524" layer="91"/>
+</segment>
 </net>
 <net name="N$7" class="0">
@@
 <segment>
 <label x="-71.12" y="43.18" size="1.778" layer="95" rot="R180" xref="yes"/>
-<pinref part="SL2" gate="G$1" pin="1"/>
-<wire x1="-64.77" y1="43.18" x2="-71.12" y2="43.18" width="0.1524" layer="91"/>
+<pinref part="SV1" gate="1" pin="1"/>
+<wire x1="-60.96" y1="43.18" x2="-71.12" y2="43.18" width="0.1524" layer="91"/>
 </segment>
 <segment>
@@
 <segment>
 <label x="-66.04" y="40.64" size="1.778" layer="95" rot="R180" xref="yes"/>
-<pinref part="SL2" gate="G$1" pin="2"/>
-<wire x1="-64.77" y1="40.64" x2="-66.04" y2="40.64" width="0.1524" layer="91"/>
+<pinref part="SV1" gate="1" pin="2"/>
+<wire x1="-60.96" y1="40.64" x2="-66.04" y2="40.64" width="0.1524" layer="91"/>
 </segment>
 <segment>
@@
 </segment>
 </net>
+<net name="N$6" class="0">
+<segment>
+<pinref part="Q8" gate="G$1" pin="B"/>
+<pinref part="R11" gate="G$1" pin="2"/>
+<wire x1="11.43" y1="-16.51" x2="8.89" y2="-16.51" width="0.1524" layer="91"/>
+</segment>
+</net>
+<net name="N$5" class="0">
+<segment>
+<pinref part="Q7" gate="G$1" pin="B"/>
+<pinref part="R10" gate="G$1" pin="2"/>
+<wire x1="-11.43" y1="-16.51" x2="-13.97" y2="-16.51" width="0.1524" layer="91"/>
+</segment>
+</net>
+<net name="N$4" class="0">
+<segment>
+<pinref part="Q6" gate="G$1" pin="B"/>
+<pinref part="R9" gate="G$1" pin="2"/>
+<wire x1="-34.29" y1="-16.51" x2="-36.83" y2="-16.51" width="0.1524" layer="91"/>
+</segment>
+</net>
+<net name="N$8" class="0">
+<segment>
+<pinref part="Q5" gate="G$1" pin="B"/>
+<pinref part="R8" gate="G$1" pin="2"/>
+<wire x1="-57.15" y1="-16.51" x2="-59.69" y2="-16.51" width="0.1524" layer="91"/>
+</segment>
+</net>
